File: kicad/tp325-meter.sch (KiCad schematic (older format))
At the start: 68 parts, among them J1 2x3-Male-Header, J2 2x3-Male-Header, U1 SA56-21SRWA, U10 SN74LS47N, U11 SN74HC595N, U12 LM324KN, U13 SA56-21SRWA, U14 SN74LS47N, U2 SN74LS47N, U3 SN74HC595N, U4 MSP430G2152IN2, U5 SA56-21SRWA, U6 SN74LS47N, U7 LM317KN, U8 LF33CV, U9 SA56-21SRWA

Commit message: partial lib/sch fix
Parts:
- removed C10, C11, C3, C4, C9: 0.1u, symbol tp325-meter:Capacitor-Nonpolar
- removed R10, R11, R12, R13, R14, R15, R18, R19, R20, R21, R24, R25, R27, R32, R33, R35, R36, R37, R38, R39, R9: 180, symbol tp325-meter:Resistor
- removed U10, U14, U6: SN74LS47N, symbol tp325-meter:SN74LS47N
- removed U11: SN74HC595N, symbol tp325-meter:SN74HC595N
- added C?: 0.1u, symbol tp325-meter:Capacitor-Nonpolar
Connections:
- net labels removed: SER
- wire segments 290 -> 227
- no-connect marks 28 -> 18
Other:
- note added: "PROTOBOARD-4"
- moved on the sheet: C2, R1, R2, R3, R4, R5, R6, R7, R8, U1, U13, U2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

Commit message: protoboard-3 schematic
Parts:
- removed R22, R23, R29, R30: 22k, symbol tp325-meter:Resistor
- removed R31: 56k, symbol tp325-meter:Resistor
- removed R34: 1.5k, symbol tp325-meter:Resistor
- removed U12: LM324KN, symbol tp325-meter:LM324KN
- added C?: 0.1u, symbol tp325-meter:Capacitor-Nonpolar
- added J?: 2x1-Header, symbol tp325-meter:2x1-Header
- added Q? (x4): TP2104, symbol tp325-meter:TP2104
- added Q? (x4): BS170, symbol tp325-meter:BS170
- added R? (x8): 1.5k, symbol tp325-meter:Resistor
- added U?: INA180A2, symbol tp325-meter:INA180A2
- R26: value 4.7 -> 8.2
- R28: value 68 -> 56
Connections:
- net labels added: DIG1, DIG2, DIG3, DIG4, PWR1, PWR2, PWR3, PWR4
- wire segments 227 -> 270
- no-connect marks 18 -> 16
Other:
- note added: "PROTOBOARD-3"
- note removed: "72R Meter Sense Voltages Relative to DC-\nVoltage Mode (6V): Vdiff=72mV, Vcmn=5.96V\nCurrent Mode (6V/6A): Vdiff=74mV, Vcmn=6.04V\n\nFirst-Stage Buffer to Eliminate Common-Mode\nSecond-Stage Gain of 38 for 2.75V Full-Scale"
- moved on the sheet: R26, R28

Commit message: updated schematic
Parts:
- removed C7: 2.2u, symbol tp325-meter:Capacitor-Nonpolar
- removed D1, D2: 1N4001, symbol tp325-meter:Diode
- removed J1, J2: 2x3-Male-Header, symbol tp325-meter:2x3-Male-Header
- added C10: 22u, symbol tp325-meter:Capacitor-Polar
- added C2: 0.1u, symbol tp325-meter:Capacitor-Nonpolar
- added C4: 1u, symbol tp325-meter:Capacitor-Nonpolar
- added C5, C7: 10u, symbol tp325-meter:Capacitor-Polar
- added C9: 100u, symbol tp325-meter:Capacitor-Polar
- added D1, D2: 1N4001, symbol tp325-meter:1N4001
- added J1: 2x1-Header, symbol tp325-meter:2x1-Header
- added Q1: 2N3904, symbol tp325-meter:2N3904
- added Q2: BS170, symbol tp325-meter:BS170
- added R1: 180k, symbol tp325-meter:Resistor
- added R2: 15k, symbol tp325-meter:Resistor
- added R3: 150k, symbol tp325-meter:Resistor
- added R6: 47k, symbol tp325-meter:Resistor
- added R7: 4.7K, symbol tp325-meter:Resistor
- added R8: 100, symbol tp325-meter:Resistor
- C1: value 0.1u -> 10n
- C6: value 10u -> 10n
- gave numbers to parts that had none: 20
- renumbered C2 to C13, C5 to C3, R26 to R13, R28 to R14, R1 to R19, R2 to R20, R3 to R21, R4 to R22, R5 to R23, R6 to R24, R8 to R25, R7 to R26, R17 to R4, R16 to R5, U7 to U1, U13 to U10, U4 to U2, U8 to U3, U3 to U4, U2 to U6, U1 to U7, U5 to U8
Connections:
- net ADC is gone; now on an unnamed net: U2.4 (P1.2)
- net RX is gone; now on an unnamed net: U2.2 (P1.0)
- net TX is gone; now on an unnamed net: U2.3 (P1.1)
- net +15V: now also D1.1 (K), J1.1 (Pin_1), R1.1, R3.2
- net +3V3: now also C1.1, C10.1, C2.1, C4.1, R6.1; no longer C1.2
- net +5V: now also C7.1, D1.2 (A), D2.1 (K); no longer C6.1
- net GND: now also C1.2, C10.2, C2.2, C4.2, C5.2, C7.2, C9.2, J1.2 (Pin_2), Q1.1 (E), Q2.3 (S), R2.2, R7.1; no longer C1.1
- net at U2.7 (P1.5): now also C8.1, C9.1, R7.2, R8.1
- net at R4.1, R5.2, U1.1 (ADJ): now also C5.1, D2.2 (A), Q2.1 (D); no longer C8.1
- net at U5.1: now also R8.2
- net MTRIN renamed MTR-
- net MTROUT renamed MTR+
- net RCLK: no longer names the net of U2.10 (P2.2)
- net SBWTCK: no longer names the net of U2.17 (TEST)
- net SBWTDIO: no longer names the net of U2.16 (~RST)
- net SBWTDIO: now also C6.1, R6.2
- net SRCLK: no longer names the net of U2.9 (P2.1)
- net ~OE: no longer names the net of U2.12 (P2.4)
- net ~SRCLR: no longer names the net of U2.11 (P2.3)
- new net: Q1.2 (B), R1.2, R2.1
- new net: Q1.3 (C), Q2.2 (G), R3.1
- no-connect marks 16 -> 20
Other:
- note added: "PROTOBOARD-1"
- note added: "PROTOBOARD-2"
- moved on the sheet: C11, C12, C13, C3, J2, R13, R14, R19, R20, R21, R22, R23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
